Commit message: change camera parent link to link1

File: ros2_ws/src/hitbot_sim/urdf/Z-Arm_10042C0_gazebo_properties.urdf.xacro (robot description, xacro)
@@ -10,5 +10,5 @@
   <xacro:include filename="$(find hitbot_sim)/urdf/Z-Arm_10042C0_gazebo.urdf" />
   <!-- IntelRealsense D435 (Plugin) -->
-  <xacro:sensor_d455 parent="link3" name="camera_1" use_nominal_extrinsics="$(arg use_nominal_extrinsics)">
+  <xacro:sensor_d455 parent="link1" name="camera_1" use_nominal_extrinsics="$(arg use_nominal_extrinsics)">
     <xacro:insert_block name="camera_1_pose" />
   </xacro:sensor_d455>

File: ros2_ws/src/hitbot_sim/urdf/sensors/d435.urdf.xacro (robot description, xacro)
@@ -56,5 +56,5 @@
         <geometry>
       <!-- <box size="${d455_cam_width} ${d455_cam_depth}  ${d455_cam_height}"/>-->
-	          <mesh filename="file://$(find realsense2_description)/meshes/d435.stl"/>
+	          <mesh filename="file://$(find realsense2_description)/meshes/d435.dae"/>
        </geometry>
         <material name="aluminum"/>
