Commit message: set camera pose x=-0.23 z=0.61 in src/scara_moveit/scara_moveit_config/config/Z-Arm_10042C0_gazebo_sensor_properties.urdf.xacro

File: ros2_ws/src/scara_moveit/scara_moveit_config/config/Z-Arm_10042C0_gazebo_sensor_properties.urdf.xacro (robot description, xacro)
@@ -4,5 +4,6 @@
   <xacro:arg name="use_nominal_extrinsics" default="true"/>
   <xacro:property name="camera_1_pose">
-    <origin xyz="0.0 0.0 0.07" rpy="0 0 0" />
+    <origin xyz="-0.23 0.0 0.61" rpy="0 0 0" />
+    -0.15609 -0.0016863 0.25062
   </xacro:property>
 </robot>
