Commit message: integrate camera_link to workld and map and odom

File: ros2_ws/src/scara_moveit/mushroom_moveit_config/config/scara_description.ros2_control.xacro (robot description, xacro)
@@ -6,5 +6,6 @@
             <hardware>
                 <!-- By default, set up controllers for simulation. This won't work on real hardware -->
-                <plugin>mock_components/GenericSystem</plugin>
+		    <plugin>scara/ScaraHardware</plugin>
+		<!--<plugin>mock_components/GenericSystem</plugin>-->
             </hardware>
             <joint name="joint1">

File: ros2_ws/src/scara_moveit/scara_description/urdf/mushroom_bot3_urdf.urdf (robot description, URDF)
Before this commit: robot scara_description, 6 links, 5 joints
Links:
- added link world
Joints:
- added joint base_joint: type fixed, parent world, child base_link, origin xyz=0 0 0 rpy=1.57 0 1.57
