Commit message: upload png of obstacle

File: ros2_ws/src/scara_moveit/scara_description/urdf/mushroom_bot3_urdf.urdf (robot description, URDF)
Before this commit: robot scara_description, 7 links, 6 joints
Joints:
- joint base_joint: origin xyz=0 0 0 rpy=1.57 0 1.57 -> xyz=0 0.6 0.0 rpy=1.57 -1.57 0.0
- joint joint2: axis 0 0 -1 -> 0 0 1
- joint joint3: axis 0 0 -1 -> 0 0 1

Commit message: update moveit config for move_to_pose test

File: ros2_ws/src/scara_moveit/scara_description/urdf/mushroom_bot3_urdf.urdf (robot description, URDF)
Before this commit: robot scara_description, 7 links, 6 joints
Joints:
- joint base_joint: origin xyz=0 0.6 0.0 rpy=1.57 -1.57 0.0 -> xyz=0 0.6 0.0 rpy=0.0 0.0 0.0
- joint joint1: limit lower=-0.15 upper=0.0 effort=5 velocity=0.01 -> lower=-0.15 upper=0.3 effort=20 velocity=1.0
- joint joint2: limit lower=-2.87 upper=2.87 effort=0.5 velocity=0.01 -> lower=-2.87 upper=2.87 effort=20 velocity=1.0
- joint joint3: limit lower=-3.1415 upper=3.1415 effort=0.5 velocity=0.01 -> lower=-3.1415 upper=3.1415 effort=20 velocity=1.0
- joint joint4: limit lower=-3.1415 upper=3.1415 effort=0.5 velocity=0.01 -> lower=-3.1415 upper=3.1415 effort=20 velocity=1.0

File: ros2_ws/src/scara_moveit/scara_moveit_config/config/mushroom_bot3_urdf.ros2_control.xacro (robot description, xacro)
@@ -6,7 +6,7 @@
             <hardware>
                 <!-- By default, set up controllers for simulation. This won't work on real hardware
+                    <plugin>scara/ScaraHardware</plugin>
+                 -->
                 <plugin>mock_components/GenericSystem</plugin>
-                 -->
-                    <plugin>scara/ScaraHardware</plugin>
             </hardware>
             <joint name="joint1">

File: ros2_ws/src/scara_moveit/scara_moveit_config/config/mushroom_bot3_urdf.urdf (robot description, URDF)
Before this commit: robot scara_description, 6 links, 5 joints
Joints:
- joint joint1: limit lower=-0.15 upper=0.0 effort=5 velocity=0.01 -> lower=-0.3 upper=0.3 effort=20 velocity=1.0
- joint joint2: limit lower=-2.87 upper=2.87 effort=0.5 velocity=0.01 -> lower=-2.87 upper=2.87 effort=20 velocity=1.0
- joint joint3: limit lower=-3.1415 upper=3.1415 effort=0.5 velocity=0.01 -> lower=-3.1415 upper=3.1415 effort=20 velocity=1.0
- joint joint4: limit lower=-3.1415 upper=3.1415 effort=0.5 velocity=0.01 -> lower=-3.1415 upper=3.1415 effort=20 velocity=1.0

File: ros2_ws/src/scara_moveit/scara_moveit_config/config/scara_description.srdf.xacro (robot description, xacro)
@@ -1,7 +1,3 @@
 <?xml version="1.0" encoding="UTF-8"?>
-<!--This does not replace URDF, and is not an extension of URDF.
-    This is a format for representing semantic information about the robot structure.
-    A URDF file must exist for this robot as well, where the joints and the links that are referenced are defined
--->
 <robot name="scara_description">
   <group name="scara_arm">

Commit message: back fromdocker mushroom_rviz2_x11

File: ros2_ws/src/scara_moveit/scara_description/urdf/mushroom_bot3_urdf.urdf (robot description, URDF)
Before this commit: robot scara_description, 7 links, 6 joints
Joints:
- joint base_joint: origin xyz=0 0.6 0.0 rpy=0.0 0.0 0.0 -> xyz=0 0.0 0.0 rpy=0.0 0.0 0.0

File: ros2_ws/src/scara_moveit/scara_moveit_config/config/mushroom_bot3_urdf.ros2_control.xacro (robot description, xacro)
@@ -6,7 +6,7 @@
             <hardware>
                 <!-- By default, set up controllers for simulation. This won't work on real hardware
+                <plugin>mock_components/GenericSystem</plugin>
+                 -->
                     <plugin>scara/ScaraHardware</plugin>
-                 -->
-                <plugin>mock_components/GenericSystem</plugin>
             </hardware>
             <joint name="joint1">

Commit message: reinstall extension to remove the offset angle=-20

File: ros2_ws/src/scara_moveit/scara_description/urdf/mushroom_bot3_urdf.urdf (robot description, URDF)
Before this commit: robot scara_description, 7 links, 6 joints
Joints:
- joint joint5: origin xyz=0.172158865969243 0 0 rpy=0 0 0 -> xyz=0.262158865969243 0 0 rpy=0 0 0

Commit message: update to yolo11

File: ros2_ws/src/scara_moveit/scara_description/urdf/mushroom_bot3_urdf.urdf (robot description, URDF)
Before this commit: robot scara_description, 7 links, 6 joints
Joints:
- joint joint1: origin xyz=0 0 0.30686 rpy=0 0 0 -> xyz=0 0 0.20686 rpy=0 0 0
- joint joint4: axis 0 0 1 -> 0 0 -1; limit lower=-3.1415 upper=3.1415 effort=20 velocity=1.0 -> lower=-1.57 upper=1.57 effort=20 velocity=1.0
